File: arduino/KiCad/arduino_wstation.sch (KiCad schematic (older format))
At the start: 44 parts, among them IC1 SHT15 breakout, IC2 BMP180 breakout, P1 Digital, P2 COM, P3 ADC, P4 Analog, P5 ADC, U1 74HC245, U2 RFM22B

Commit message: Update arduino schematics. Add final code
Connections:
- net labels added: AN7
- net labels removed: AN6
- wire segments 203 -> 204
Other:
- note added: "North direction = Support arm"
- note added: "Reed relay (1 pulse/rev = 0.345708m/rev)"
- note removed: "North direction = support arm:"
- note removed: "Reed relay"
