File: arduino/KiCad/arduino_wstation_rfm69.sch (KiCad schematic (older format))
At the start: 44 parts, among them IC1 SHT15 breakout, IC2 BMP180 breakout, P1 Digital, P2 COM, P3 ADC, P4 Analog, P5 ADC, U1 74HC245, U2 RFM69HCW

Commit message: Update Arduino-RFM22B and Arduino-RFM69 schematics files
Parts:
- 1Q2, 1Q3, 1Q4, 1Q5: symbol arduino_wstation-rescue:OPTO_NPN-wstation-cache -> arduino_wstation_rfm69-rescue:OPTO_NPN-wstation-cache-arduino_wstation-rescue
- IC1: symbol arduino_wstation-rescue:SHT1X-sht10_11_15 -> arduino_wstation_rfm69-rescue:SHT1X-sht10_11_15-arduino_wstation-rescue
- IC2: symbol arduino_wstation-rescue:BMP180-bmp180 -> arduino_wstation_rfm69-rescue:BMP180-bmp180-arduino_wstation-rescue
- P1, P4: symbol arduino_wstation-rescue:CONN_12-wstation-cache -> arduino_wstation_rfm69-rescue:CONN_12-wstation-cache-arduino_wstation-rescue
- P2: symbol arduino_wstation-rescue:CONN_6-wstation-cache -> arduino_wstation_rfm69-rescue:CONN_6-wstation-cache-arduino_wstation-rescue
- P3, P5: symbol arduino_wstation-rescue:CONN_2-wstation-cache -> arduino_wstation_rfm69-rescue:CONN_2-wstation-cache-arduino_wstation-rescue
- U2: symbol arduino_wstation-rescue:RFM69HCW -> arduino_wstation_rfm69-rescue:RFM69HCW-arduino_wstation-rescue
Changed lines of the file:
@@
 EESchema Schematic File Version 4
-LIBS:arduino_wstation-cache
+LIBS:arduino_wstation_rfm69-cache
 EELAYER 30 0
 EELAYER END
@@
 $EndDescr
 $Comp
-L arduino_wstation-rescue:CONN_12-wstation-cache P1
+L arduino_wstation_rfm69-rescue:CONN_12-wstation-cache-arduino_wstation-rescue P1
 U 1 1 552014A1
 P 6725 2375
@@
 $EndComp
 $Comp
-L arduino_wstation-rescue:CONN_12-wstation-cache P4
+L arduino_wstation_rfm69-rescue:CONN_12-wstation-cache-arduino_wstation-rescue P4
 U 1 1 552014EF
 P 7050 2375
@@
 A3
 $Comp
-L arduino_wstation-rescue:CONN_2-wstation-cache P3
+L arduino_wstation_rfm69-rescue:CONN_2-wstation-cache-arduino_wstation-rescue P3
 U 1 1 55201A4F
 P 6675 3200
@@
 Shield Arduino Pro Mini \n
 $Comp
-L arduino_wstation-rescue:CONN_2-wstation-cache P5
+L arduino_wstation_rfm69-rescue:CONN_2-wstation-cache-arduino_wstation-rescue P5
 U 1 1 552112EB
 P 7100 3200
@@
 A6
 $Comp
-L arduino_wstation-rescue:BMP180-bmp180 IC2
+L arduino_wstation_rfm69-rescue:BMP180-bmp180-arduino_wstation-rescue IC2
 U 1 1 58010E86
 P 10025 5775
@@
 $EndComp
 $Comp
-L arduino_wstation-rescue:RFM69HCW U2
+L arduino_wstation_rfm69-rescue:RFM69HCW-arduino_wstation-rescue U2
 U 1 1 58011353
 P 10000 2725
@@
 $EndComp
 $Comp
-L arduino_wstation-rescue:OPTO_NPN-wstation-cache 1Q2
+L arduino_wstation_rfm69-rescue:OPTO_NPN-wstation-cache-arduino_wstation-rescue 1Q2
 U 1 1 5801EB4C
 P 2625 6600
@@
 $EndComp
 $Comp
-L arduino_wstation-rescue:OPTO_NPN-wstation-cache 1Q3
+L arduino_wstation_rfm69-rescue:OPTO_NPN-wstation-cache-arduino_wstation-rescue 1Q3
 U 1 1 5801EBFA
 P 3500 6600
@@
 $EndComp
 $Comp
-L arduino_wstation-rescue:OPTO_NPN-wstation-cache 1Q4
+L arduino_wstation_rfm69-rescue:OPTO_NPN-wstation-cache-arduino_wstation-rescue 1Q4
 U 1 1 5801ED94
 P 4350 6600
@@
 	1700 6800 5275 6800
 $Comp
-L arduino_wstation-rescue:SHT1X-sht10_11_15 IC1
+L arduino_wstation_rfm69-rescue:SHT1X-sht10_11_15-arduino_wstation-rescue IC1
 U 1 1 58010BB1
 P 10000 4625
@@
 $EndComp
 $Comp
-L arduino_wstation-rescue:CONN_6-wstation-cache P2
+L arduino_wstation_rfm69-rescue:CONN_6-wstation-cache-arduino_wstation-rescue P2
 U 1 1 55201543
 P 6875 1575
@@
 	2925 6125 3800 6125
 $Comp
-L arduino_wstation-rescue:OPTO_NPN-wstation-cache 1Q5
+L arduino_wstation_rfm69-rescue:OPTO_NPN-wstation-cache-arduino_wstation-rescue 1Q5
 U 1 1 5801EE37
 P 5175 6600
