File: arduino/KiCad/arduino_ftdi/arduino_ftdi.sch (KiCad schematic (older format))
At the start: 23 parts, among them J1 RJ45, J10 9V-12V, J11 3V3 & 5V, J12 9V-12V, J13 3V3 & 5V, J2 IN/OUT, J3 DTR/TX/RX, J4 Power output 3V3, J5 NC, J6 DTR-FTDI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

Commit message: Update ftdi interfaces (remove the unnecesary load resistors)
Parts:
- removed R1, R3: R120, symbol Device:R
- renumbered R2 to R1, R4 to R2
Connections:
- wire segments 145 -> 138
Changed lines of the file:
@@
 Sheet 1 1
 Title "RS422 5V to UART 3V3 interface"
-Date "2021-03-06"
-Rev "2.2"
+Date "2021-04-11"
+Rev "2.3"
 Comp ""
 Comment1 "Interface to provide UART from RS442 on Ethernet cable"
@@
 Wire Wire Line
 	5250 1525 5250 1475
-Wire Wire Line
-	5250 1475 5550 1475
 $Comp
 L Interface_UART:MAX488E U2
@@
 	5150 2550 5150 2500
 Wire Wire Line
-	5150 2500 5250 2500
-Wire Wire Line
 	5200 2650 5200 2600
 Wire Wire Line
-	5200 2600 5550 2600
-Wire Wire Line
 	5150 2850 5150 2900
 Wire Wire Line
@@
 $Comp
 L Device:R R1
-U 1 1 5F62DFF3
-P 5400 1275
-F 0 "R1" V 5193 1275 50  0000 C CNN
-F 1 "R120" V 5284 1275 50  0000 C CNN
-F 2 "" V 5330 1275 50  0001 C CNN
-F 3 "~" H 5400 1275 50  0001 C CNN
-	1    5400 1275
-	0    1    1    0
-$EndComp
-$Comp
-L Device:R R2
 U 1 1 5F62DFF4
 P 5400 2050
-F 0 "R2" V 5193 2050 50  0000 C CNN
+F 0 "R1" V 5193 2050 50  0000 C CNN
 F 1 "R120" V 5284 2050 50  0000 C CNN
 F 2 "" V 5330 2050 50  0001 C CNN
@@
 $EndComp
 $Comp
-L Device:R R3
-U 1 1 5F62DFF5
-P 5400 2375
-F 0 "R3" V 5193 2375 50  0000 C CNN
-F 1 "R120" V 5284 2375 50  0000 C CNN
-F 2 "" V 5330 2375 50  0001 C CNN
-F 3 "~" H 5400 2375 50  0001 C CNN
-	1    5400 2375
-	0    1    1    0
-$EndComp
-$Comp
-L Device:R R4
+L Device:R R2
 U 1 1 5F62DFF6
 P 5400 3175
-F 0 "R4" V 5193 3175 50  0000 C CNN
+F 0 "R2" V 5193 3175 50  0000 C CNN
 F 1 "R120" V 5284 3175 50  0000 C CNN
 F 2 "" V 5330 3175 50  0001 C CNN
@@
 $EndComp
 Wire Wire Line
-	5550 1275 5550 1475
-Connection ~ 5550 1475
-Wire Wire Line
-	5550 1475 5625 1475
-Wire Wire Line
-	5250 1275 5250 1375
-Connection ~ 5250 1375
-Wire Wire Line
 	5250 1375 5625 1375
 Wire Wire Line
@@
 	5250 1425 5250 1375
 Wire Wire Line
-	5550 2375 5550 2600
-Connection ~ 5550 2600
-Wire Wire Line
-	5550 2600 5625 2600
-Wire Wire Line
-	5250 2375 5250 2500
-Connection ~ 5250 2500
-Wire Wire Line
-	5250 2500 5625 2500
-Wire Wire Line
 	5550 3175 5550 2800
 Connection ~ 5550 2800
@@
 Text Label 7025 2800 0    51   ~ 0
 TX-FTDI
+Wire Wire Line
+	5250 1475 5625 1475
+Wire Wire Line
+	5200 2600 5625 2600
+Wire Wire Line
+	5150 2500 5625 2500
 $EndSCHEMATC
