File: arduino/KiCad/arduino_ftdi/usb_ftdi.sch (KiCad schematic (older format))
At the start: 9 parts, among them J1 RJ45, J2 IN, U1 MAX488E, U2 MAX488E

Commit message: Update ftdi interfaces (remove the unnecesary load resistors)
Parts:
- removed R2, R4: R120, symbol Device:R
- renumbered R3 to R2
Connections:
- wire segments 72 -> 64
Changed lines of the file:
@@
 Sheet 1 1
 Title "USB-UART to RS422 5V interface"
-Date "2021-03-06"
-Rev "1.1"
+Date "2021-04-11"
+Rev "1.3"
 Comp ""
 Comment1 "Interface from UART to RS442 on Ethernet cable"
@@
 	4950 3450 4950 3250
 Wire Wire Line
-	5725 2950 5350 2950
-Connection ~ 5725 2950
-Wire Wire Line
-	5725 3225 5725 2950
-Wire Wire Line
-	5425 2850 5350 2850
-Connection ~ 5425 2850
-Wire Wire Line
-	5425 3225 5425 2850
-Wire Wire Line
 	5725 2550 5350 2550
 Connection ~ 5725 2550
@@
 	5950 1425 5725 1425
 Wire Wire Line
-	5725 1825 5350 1825
-Connection ~ 5725 1825
-Wire Wire Line
-	5725 2100 5725 1825
-Wire Wire Line
-	5425 1725 5350 1725
-Connection ~ 5425 1725
-Wire Wire Line
-	5425 2100 5425 1725
-Wire Wire Line
 	5725 1425 5350 1425
 Connection ~ 5725 1425
@@
 	5425 1325 5425 1525
 $Comp
-L Device:R R4
-U 1 1 5F664FC1
-P 5575 3225
-F 0 "R4" V 5368 3225 50  0000 C CNN
-F 1 "R120" V 5459 3225 50  0000 C CNN
-F 2 "" V 5505 3225 50  0001 C CNN
-F 3 "~" H 5575 3225 50  0001 C CNN
-	1    5575 3225
-	0    -1   1    0
-$EndComp
-$Comp
-L Device:R R3
+L Device:R R2
 U 1 1 5F664745
 P 5575 2425
-F 0 "R3" V 5368 2425 50  0000 C CNN
+F 0 "R2" V 5368 2425 50  0000 C CNN
 F 1 "R120" V 5459 2425 50  0000 C CNN
 F 2 "" V 5505 2425 50  0001 C CNN
@@
 $EndComp
 $Comp
-L Device:R R2
-U 1 1 5F663EB7
-P 5575 2100
-F 0 "R2" V 5368 2100 50  0000 C CNN
-F 1 "R120" V 5459 2100 50  0000 C CNN
-F 2 "" V 5505 2100 50  0001 C CNN
-F 3 "~" H 5575 2100 50  0001 C CNN
-	1    5575 2100
-	0    -1   1    0
-$EndComp
-$Comp
 L Device:R R1
 U 1 1 5F6632F6
@@
 $EndComp
 Wire Wire Line
-	5725 1825 8525 1825
-Wire Wire Line
-	5425 1725 8450 1725
-Wire Wire Line
 	5725 2550 7025 2550
 Wire Wire Line
 	5425 2650 7125 2650
-Wire Wire Line
-	5425 2850 7300 2850
 Text Notes 6100 1500 2    50   ~ 0
 nc
@@
 	8250 2950 8250 2775
 Wire Wire Line
-	5725 2950 8250 2950
+	5350 1825 8525 1825
+Wire Wire Line
+	5350 1725 8450 1725
+Wire Wire Line
+	5350 2950 8250 2950
+Wire Wire Line
+	5350 2850 7300 2850
 $EndSCHEMATC

Commit message: Update FTDI interface schematics
Parts:
- removed R5: R100, symbol Device:R
- R1, R2: value R120 -> R100
Connections:
- wire segments 64 -> 63
Changed lines of the file:
@@
 EESchema Schematic File Version 4
-LIBS:usb_ftdi-cache
 EELAYER 30 0
 EELAYER END
@@
 encoding utf-8
 Sheet 1 1
-Title "USB-UART to RS422 5V interface"
-Date "2021-04-11"
-Rev "1.3"
+Title "USB-UART to RS485 5V interface"
+Date "2021-08-21"
+Rev "1.5"
 Comp ""
-Comment1 "Interface from UART to RS442 on Ethernet cable"
+Comment1 "Interface from UART to RS485 on Ethernet cable"
 Comment2 ""
 Comment3 ""
@@
 P 5575 2425
 F 0 "R2" V 5368 2425 50  0000 C CNN
-F 1 "R120" V 5459 2425 50  0000 C CNN
+F 1 "R100" V 5459 2425 50  0000 C CNN
 F 2 "" V 5505 2425 50  0001 C CNN
 F 3 "~" H 5575 2425 50  0001 C CNN
@@
 P 5575 1325
 F 0 "R1" V 5368 1325 50  0000 C CNN
-F 1 "R120" V 5459 1325 50  0000 C CNN
+F 1 "R100" V 5459 1325 50  0000 C CNN
 F 2 "" V 5505 1325 50  0001 C CNN
 F 3 "~" H 5575 1325 50  0001 C CNN
@@
 Wire Bus Line
 	2025 2125 1325 2125
-$Comp
-L Device:R R5
-U 1 1 5F70F0B5
-P 4950 3700
-F 0 "R5" V 4743 3700 50  0000 C CNN
-F 1 "R100" V 4834 3700 50  0000 C CNN
-F 2 "" V 4880 3700 50  0001 C CNN
-F 3 "~" H 4950 3700 50  0001 C CNN
-	1    4950 3700
-	-1   0    0    -1
-$EndComp
-Wire Wire Line
-	4950 3550 4950 3450
 Connection ~ 4950 3450
-Wire Wire Line
-	4950 3850 4950 4125
 Connection ~ 4950 4125
 Text Notes 1450 1350 0    51   ~ 0
@@
 Wire Wire Line
 	5350 2850 7300 2850
+Wire Wire Line
+	4950 3450 4950 4125
 $EndSCHEMATC
